File: hardware/sneak100_main_board/motors.sch (KiCad schematic (older format))
At the start: 0 parts

Commit message: motors circuit scheme
Parts:
- added C10, C3, C4, C5, C6, C7, C8, C9: 100nF, Capacitor_SMD:C_0805_2012Metric, symbol Device:C
- added J3, J4, J5, J6: Conn_01x06, Connector_PinHeader_2.54mm:PinHeader_1x06_P2.54mm_Vertical, symbol Connector_Generic:Conn_01x06
- added U1, U2, U3, U4: DRV8835, Package_SON:WSON-12-1EP_3x2mm_P0.5mm_EP1x2.65_ThermalVias, symbol Sneak100_kicad:DRV8835
Connections:
- new net +3V3: C3.1, C5.1, C7.1, C9.1, J3.4 (Pin_4), J4.4 (Pin_4), J5.4 (Pin_4), J6.4 (Pin_4), U1.12 (VCC), U2.12 (VCC), U3.12 (VCC), U4.12 (VCC)
- new net GND: C10.2, C3.2, C4.2, C5.2, C6.2, C7.2, C8.2, C9.2, J3.1 (Pin_1), J4.1 (Pin_1), J5.1 (Pin_1), J6.1 (Pin_1), U1.11 (MODE), U1.13 (Theraml_Pad), U1.6 (GND), U2.11 (MODE), U2.13 (Theraml_Pad), U2.6 (GND), U3.11 (MODE), U3.13 (Theraml_Pad), U3.6 (GND), U4.11 (MODE), U4.13 (Theraml_Pad), U4.6 (GND)
- new net LB_A: J5.3 (Pin_3)
- new net LB_B: J5.2 (Pin_2)
- new net LB_IN1: U3.10 (AIN1/APHASE), U3.8 (BIN1/BPHASE)
- new net LB_IN2: U3.7 (BIN2/BENBL), U3.9 (AIN2/AENBL)
- new net LB_OUT1: J5.6 (Pin_6), U3.2 (AOUT1), U3.4 (BOUT1)
- new net LB_OUT2: J5.5 (Pin_5), U3.3 (AOUT2), U3.5 (BOUT2)
- new net LF_A: J3.3 (Pin_3)
- new net LF_B: J3.2 (Pin_2)
- new net LF_IN1: U1.10 (AIN1/APHASE), U1.8 (BIN1/BPHASE)
- new net LF_IN2: U1.7 (BIN2/BENBL), U1.9 (AIN2/AENBL)
- new net LF_OUT1: J3.6 (Pin_6), U1.2 (AOUT1), U1.4 (BOUT1)
- new net LF_OUT2: J3.5 (Pin_5), U1.3 (AOUT2), U1.5 (BOUT2)
- new net RB_A: J6.3 (Pin_3)
- new net RB_B: J6.2 (Pin_2)
- new net RB_IN1: U4.10 (AIN1/APHASE), U4.8 (BIN1/BPHASE)
- new net RB_IN2: U4.7 (BIN2/BENBL), U4.9 (AIN2/AENBL)
- new net RB_OUT1: J6.6 (Pin_6), U4.2 (AOUT1), U4.4 (BOUT1)
- new net RB_OUT2: J6.5 (Pin_5), U4.3 (AOUT2), U4.5 (BOUT2)
- new net RF_A: J4.3 (Pin_3)
- new net RF_B: J4.2 (Pin_2)
- new net RF_IN1: U2.10 (AIN1/APHASE), U2.8 (BIN1/BPHASE)
- new net RF_IN2: U2.7 (BIN2/BENBL), U2.9 (AIN2/AENBL)
- new net RF_OUT1: J4.6 (Pin_6), U2.2 (AOUT1), U2.4 (BOUT1)
- new net RF_OUT2: J4.5 (Pin_5), U2.3 (AOUT2), U2.5 (BOUT2)
- new net VIN: C10.1, C4.1, C6.1, C8.1, U1.1 (VM), U2.1 (VM), U3.1 (VM), U4.1 (VM)
Other:
- note added: "H-Bridge control mode:\nMODE = LOW -> IN/IN\nMODE = HIGH -> PHASE/ENBL"
- note added: "Left-Back motor"
- note added: "Left-Front motor"
- note added: "Right-Back motor"
- note added: "Right-Front motor"
