File: hardware/sneak100_main_board/motors.sch (KiCad schematic (older format))
At the start: 20 parts, among them J1 Conn_01x06, J2 Conn_01x06, J3 Conn_01x06, J4 Conn_01x06, U1 DRV8835, U2 DRV8835, U3 DRV8835, U4 DRV8835

Commit message: Bigger tantalum capacitors
Parts:
- C12, C3, C6, C9: value 47uF -> 47uF/20V; footprint Capacitor_Tantalum_SMD:CP_EIA-3216-18_Kemet-A -> Capacitor_Tantalum_SMD:CP_EIA-7343-31_Kemet-D
Changed lines of the file:
@@
 AR Path="/60E0499A/610E5A56" Ref="C3"  Part="1"
 F 0 "C3" H 2468 1696 50  0000 L CNN
-F 1 "47uF" H 2468 1605 50  0000 L CNN
-F 2 "Capacitor_Tantalum_SMD:CP_EIA-3216-18_Kemet-A" H 2388 1500 50  0001 C CNN
+F 1 "47uF/20V" H 2468 1605 50  0000 L CNN
+F 2 "Capacitor_Tantalum_SMD:CP_EIA-7343-31_Kemet-D" H 2388 1500 50  0001 C CNN
 F 3 "~" H 2350 1650 50  0001 C CNN
 	1    2350 1650
@@
 AR Path="/60E0499A/61105193" Ref="C6"  Part="1"
 F 0 "C6" H 7168 1696 50  0000 L CNN
-F 1 "47uF" H 7168 1605 50  0000 L CNN
-F 2 "Capacitor_Tantalum_SMD:CP_EIA-3216-18_Kemet-A" H 7088 1500 50  0001 C CNN
+F 1 "47uF/20V" H 7168 1605 50  0000 L CNN
+F 2 "Capacitor_Tantalum_SMD:CP_EIA-7343-31_Kemet-D" H 7088 1500 50  0001 C CNN
 F 3 "~" H 7050 1650 50  0001 C CNN
 	1    7050 1650
@@
 AR Path="/60E0499A/6111802D" Ref="C9"  Part="1"
 F 0 "C9" H 2368 4596 50  0000 L CNN
-F 1 "47uF" H 2368 4505 50  0000 L CNN
-F 2 "Capacitor_Tantalum_SMD:CP_EIA-3216-18_Kemet-A" H 2288 4400 50  0001 C CNN
+F 1 "47uF/20V" H 2368 4505 50  0000 L CNN
+F 2 "Capacitor_Tantalum_SMD:CP_EIA-7343-31_Kemet-D" H 2288 4400 50  0001 C CNN
 F 3 "~" H 2250 4550 50  0001 C CNN
 	1    2250 4550
@@
 AR Path="/60E0499A/6112876D" Ref="C12"  Part="1"
 F 0 "C12" H 7168 4646 50  0000 L CNN
-F 1 "47uF" H 7168 4555 50  0000 L CNN
-F 2 "Capacitor_Tantalum_SMD:CP_EIA-3216-18_Kemet-A" H 7088 4450 50  0001 C CNN
+F 1 "47uF/20V" H 7168 4555 50  0000 L CNN
+F 2 "Capacitor_Tantalum_SMD:CP_EIA-7343-31_Kemet-D" H 7088 4450 50  0001 C CNN
 F 3 "~" H 7050 4600 50  0001 C CNN
 	1    7050 4600
