File: hardware/sneak100_main_board/lineSennsors.sch (KiCad schematic (older format))
At the start: 4 parts, among them J10 Conn_01x03, J7 Conn_01x03, J8 Conn_01x03, J9 Conn_01x03

Commit message: PCB first full layout
Parts:
- renumbered J7 to J6, J8 to J7, J9 to J8, J10 to J9
Changed lines of the file:
@@
 $EndDescr
 $Comp
-L Connector_Generic:Conn_01x03 J7
+L Connector_Generic:Conn_01x03 J6
 U 1 1 60E05377
 P 4050 2550
-F 0 "J7" H 4130 2592 50  0000 L CNN
+F 0 "J6" H 4130 2592 50  0000 L CNN
 F 1 "Conn_01x03" H 4130 2501 50  0000 L CNN
 F 2 "Connector_PinHeader_2.54mm:PinHeader_1x03_P2.54mm_Vertical" H 4050 2550 50  0001 C CNN
@@
 $EndComp
 $Comp
-L Connector_Generic:Conn_01x03 J8
+L Connector_Generic:Conn_01x03 J7
 U 1 1 60E06B30
 P 4050 2950
-F 0 "J8" H 4130 2992 50  0000 L CNN
+F 0 "J7" H 4130 2992 50  0000 L CNN
 F 1 "Conn_01x03" H 4130 2901 50  0000 L CNN
 F 2 "Connector_PinHeader_2.54mm:PinHeader_1x03_P2.54mm_Vertical" H 4050 2950 50  0001 C CNN
@@
 $EndComp
 $Comp
-L Connector_Generic:Conn_01x03 J9
+L Connector_Generic:Conn_01x03 J8
 U 1 1 60E07495
 P 4050 3350
-F 0 "J9" H 4130 3392 50  0000 L CNN
+F 0 "J8" H 4130 3392 50  0000 L CNN
 F 1 "Conn_01x03" H 4130 3301 50  0000 L CNN
 F 2 "Connector_PinHeader_2.54mm:PinHeader_1x03_P2.54mm_Vertical" H 4050 3350 50  0001 C CNN
@@
 $EndComp
 $Comp
-L Connector_Generic:Conn_01x03 J10
+L Connector_Generic:Conn_01x03 J9
 U 1 1 60E07950
 P 4050 3750
-F 0 "J10" H 4130 3792 50  0000 L CNN
+F 0 "J9" H 4130 3792 50  0000 L CNN
 F 1 "Conn_01x03" H 4130 3701 50  0000 L CNN
 F 2 "Connector_PinHeader_2.54mm:PinHeader_1x03_P2.54mm_Vertical" H 4050 3750 50  0001 C CNN
@@
 $EndComp
 $Comp
-L power:+3.3V #PWR075
+L power:+3.3V #PWR076
 U 1 1 60E08D03
 P 3850 2550
-F 0 "#PWR075" H 3850 2400 50  0001 C CNN
+F 0 "#PWR076" H 3850 2400 50  0001 C CNN
 F 1 "+3.3V" V 3865 2678 50  0000 L CNN
 F 2 "" H 3850 2550 50  0001 C CNN
@@
 $EndComp
 $Comp
-L power:+3.3V #PWR077
+L power:+3.3V #PWR078
 U 1 1 60E097F5
 P 3850 2950
-F 0 "#PWR077" H 3850 2800 50  0001 C CNN
+F 0 "#PWR078" H 3850 2800 50  0001 C CNN
 F 1 "+3.3V" V 3865 3078 50  0000 L CNN
 F 2 "" H 3850 2950 50  0001 C CNN
@@
 $EndComp
 $Comp
-L power:+3.3V #PWR079
+L power:+3.3V #PWR080
 U 1 1 60E09BF6
 P 3850 3350
-F 0 "#PWR079" H 3850 3200 50  0001 C CNN
+F 0 "#PWR080" H 3850 3200 50  0001 C CNN
 F 1 "+3.3V" V 3865 3478 50  0000 L CNN
 F 2 "" H 3850 3350 50  0001 C CNN
@@
 $EndComp
 $Comp
-L power:+3.3V #PWR081
+L power:+3.3V #PWR082
 U 1 1 60E0A09F
 P 3850 3750
-F 0 "#PWR081" H 3850 3600 50  0001 C CNN
+F 0 "#PWR082" H 3850 3600 50  0001 C CNN
 F 1 "+3.3V" V 3865 3878 50  0000 L CNN
 F 2 "" H 3850 3750 50  0001 C CNN
@@
 $EndComp
 $Comp
-L power:GND #PWR080
+L power:GND #PWR081
 U 1 1 60E0A641
 P 3850 3650
-F 0 "#PWR080" H 3850 3400 50  0001 C CNN
+F 0 "#PWR081" H 3850 3400 50  0001 C CNN
 F 1 "GND" V 3855 3522 50  0000 R CNN
 F 2 "" H 3850 3650 50  0001 C CNN
@@
 $EndComp
 $Comp
-L power:GND #PWR078
+L power:GND #PWR079
 U 1 1 60E0ADFF
 P 3850 3250
-F 0 "#PWR078" H 3850 3000 50  0001 C CNN
+F 0 "#PWR079" H 3850 3000 50  0001 C CNN
 F 1 "GND" V 3855 3122 50  0000 R CNN
 F 2 "" H 3850 3250 50  0001 C CNN
@@
 $EndComp
 $Comp
-L power:GND #PWR076
+L power:GND #PWR077
 U 1 1 60E0B1BF
 P 3850 2850
-F 0 "#PWR076" H 3850 2600 50  0001 C CNN
+F 0 "#PWR077" H 3850 2600 50  0001 C CNN
 F 1 "GND" V 3855 2722 50  0000 R CNN
 F 2 "" H 3850 2850 50  0001 C CNN
@@
 $EndComp
 $Comp
-L power:GND #PWR074
+L power:GND #PWR075
 U 1 1 60E0B57F
 P 3850 2450
-F 0 "#PWR074" H 3850 2200 50  0001 C CNN
+F 0 "#PWR075" H 3850 2200 50  0001 C CNN
 F 1 "GND" V 3855 2322 50  0000 R CNN
 F 2 "" H 3850 2450 50  0001 C CNN
