File: hardware/sneak100_main_board/lineSennsors.sch (KiCad schematic (older format))
At the start: 4 parts, among them J6 Conn_01x03, J7 Conn_01x03, J8 Conn_01x03, J9 Conn_01x03

Commit message: bluetooth en & status connection
Other:
- note added: "4x QTR-1A"
- note added: "Line sensors"
- note removed: "QTR-1A sensors connection"
Changed lines of the file:
@@
 Text HLabel 3850 3850 0    50   Output ~ 0
 READ_RR
-Text Notes 2950 2150 0    100  ~ 20
-QTR-1A sensors connection
+Text Notes 3550 1800 0    100  ~ 20
+Line sensors
+Text Notes 3800 2000 0    50   ~ 10
+4x QTR-1A
 $EndSCHEMATC

Commit message: proximity sensors connectors
Parts:
- J6, J7, J8, J9: footprint Connector_PinHeader_2.54mm:PinHeader_1x03_P2.54mm_Vertical -> Connector_PinSocket_2.54mm:PinSocket_1x03_P2.54mm_Vertical
Changed lines of the file:
@@
 F 0 "J6" H 4130 2592 50  0000 L CNN
 F 1 "Conn_01x03" H 4130 2501 50  0000 L CNN
-F 2 "Connector_PinHeader_2.54mm:PinHeader_1x03_P2.54mm_Vertical" H 4050 2550 50  0001 C CNN
+F 2 "Connector_PinSocket_2.54mm:PinSocket_1x03_P2.54mm_Vertical" H 4050 2550 50  0001 C CNN
 F 3 "~" H 4050 2550 50  0001 C CNN
 	1    4050 2550
@@
 F 0 "J7" H 4130 2992 50  0000 L CNN
 F 1 "Conn_01x03" H 4130 2901 50  0000 L CNN
-F 2 "Connector_PinHeader_2.54mm:PinHeader_1x03_P2.54mm_Vertical" H 4050 2950 50  0001 C CNN
+F 2 "Connector_PinSocket_2.54mm:PinSocket_1x03_P2.54mm_Vertical" H 4050 2950 50  0001 C CNN
 F 3 "~" H 4050 2950 50  0001 C CNN
 	1    4050 2950
@@
 F 0 "J8" H 4130 3392 50  0000 L CNN
 F 1 "Conn_01x03" H 4130 3301 50  0000 L CNN
-F 2 "Connector_PinHeader_2.54mm:PinHeader_1x03_P2.54mm_Vertical" H 4050 3350 50  0001 C CNN
+F 2 "Connector_PinSocket_2.54mm:PinSocket_1x03_P2.54mm_Vertical" H 4050 3350 50  0001 C CNN
 F 3 "~" H 4050 3350 50  0001 C CNN
 	1    4050 3350
@@
 F 0 "J9" H 4130 3792 50  0000 L CNN
 F 1 "Conn_01x03" H 4130 3701 50  0000 L CNN
-F 2 "Connector_PinHeader_2.54mm:PinHeader_1x03_P2.54mm_Vertical" H 4050 3750 50  0001 C CNN
+F 2 "Connector_PinSocket_2.54mm:PinSocket_1x03_P2.54mm_Vertical" H 4050 3750 50  0001 C CNN
 F 3 "~" H 4050 3750 50  0001 C CNN
 	1    4050 3750
