File: hardware/sneak100_main_board/power.sch (KiCad schematic (older format))
At the start: 19 parts, among them J5 Conn_01x02, Q1 AO4407, Q2 AO4407, SW1 SW_Push_SPDT, U5 LM1117-3.3, U6 S9V11F5

Commit message: Add external proximity sensor, erase old from schematic
Parts:
- removed C14: 780uF, Capacitor_THT:CP_Radial_D10.0mm_P5.00mm, symbol Device:CP
- R4: value 16k -> 18k
- renumbered C9 to C13, C10 to C14, C11 to C15, C12 to C16, C13 to C17
Other:
- note added: "Voltage divider calculations:\n\nU_in max = 8.4V\nU_out max = 3V\n\nU_out = U_in * R2/(R1+R2)\nU_out * (R1+R2) = U_in * R2\nU_out * R1+ U_out * R2 = U_in * R2\nU_out * R1 = (U_in - U_out) * R2\nR1 = R2 * (U_in - U_out)/U_out\n\nassume R2 = 10k\n\nR1 = 10000 * (8.4 - 3)/3 = 18 kohm\n"
- note removed: "Voltage divider calculations:\n\nU_in max = 8.4V\nU_out max = 3.3V\n\nU_out = U_in * R2/(R1+R2)\nU_out * (R1+R2) = U_in * R2\nU_out * R1+ U_out * R2 = U_in * R2\nU_out * R1 = (U_in - U_out) * R2\nR1 = R2 * (U_in - U_out)/U_out\n\nassume R2 = 10k\n\nR1 = 10000 * (8.4 - 3.3)/3.3 = 15454 ohm -> 16kohm\n"
Changed lines of the file:
@@
 $EndComp
 $Comp
-L power:GND #PWR048
+L power:GND #PWR051
 U 1 1 60F07A92
 P 9550 4800
-F 0 "#PWR048" H 9550 4550 50  0001 C CNN
+F 0 "#PWR051" H 9550 4550 50  0001 C CNN
 F 1 "GND" H 9555 4627 50  0000 C CNN
 F 2 "" H 9550 4800 50  0001 C CNN
@@
 $EndComp
 $Comp
-L power:+3.3V #PWR047
+L power:+3.3V #PWR050
 U 1 1 60F07C02
 P 9550 4200
-F 0 "#PWR047" H 9550 4050 50  0001 C CNN
+F 0 "#PWR050" H 9550 4050 50  0001 C CNN
 F 1 "+3.3V" H 9565 4373 50  0000 C CNN
 F 2 "" H 9550 4200 50  0001 C CNN
@@
 P 6500 4350
 F 0 "R4" H 6570 4396 50  0000 L CNN
-F 1 "16k" H 6570 4305 50  0000 L CNN
+F 1 "18k" H 6570 4305 50  0000 L CNN
 F 2 "Resistor_SMD:R_0603_1608Metric" V 6430 4350 50  0001 C CNN
 F 3 "~" H 6500 4350 50  0001 C CNN
@@
 $EndComp
 $Comp
-L power:GND #PWR049
+L power:GND #PWR052
 U 1 1 60F10E65
 P 6500 4900
-F 0 "#PWR049" H 6500 4650 50  0001 C CNN
+F 0 "#PWR052" H 6500 4650 50  0001 C CNN
 F 1 "GND" H 6505 4727 50  0000 C CNN
 F 2 "" H 6500 4900 50  0001 C CNN
@@
 	2950 2350 3100 2350
 $Comp
-L power:GND #PWR045
+L power:GND #PWR048
 U 1 1 60F76C10
 P 2050 2950
-F 0 "#PWR045" H 2050 2700 50  0001 C CNN
+F 0 "#PWR048" H 2050 2700 50  0001 C CNN
 F 1 "GND" H 2055 2777 50  0000 C CNN
 F 2 "" H 2050 2950 50  0001 C CNN
@@
 $EndComp
 $Comp
-L power:GND #PWR046
+L power:GND #PWR049
 U 1 1 60F78854
 P 2800 3500
-F 0 "#PWR046" H 2800 3250 50  0001 C CNN
+F 0 "#PWR049" H 2800 3250 50  0001 C CNN
 F 1 "GND" H 2805 3327 50  0000 C CNN
 F 2 "" H 2800 3500 50  0001 C CNN
@@
 	2800 3450 2850 3450
 $Comp
-L power:GND #PWR036
+L power:GND #PWR040
 U 1 1 60F7A03D
 P 1550 2500
-F 0 "#PWR036" H 1550 2250 50  0001 C CNN
+F 0 "#PWR040" H 1550 2250 50  0001 C CNN
 F 1 "GND" H 1555 2327 50  0000 C CNN
 F 2 "" H 1550 2500 50  0001 C CNN
@@
 Wire Wire Line
 	1550 2450 1550 2500
-Text GLabel 4150 2350 2    50   Input ~ 0
+Text GLabel 3650 2350 2    50   Input ~ 0
 SUPPLY
 Wire Wire Line
@@
 $EndComp
 $Comp
-L Device:C C10
+L Device:C C14
 U 1 1 6104BD36
 P 8800 2450
-F 0 "C10" H 8450 2500 50  0000 L CNN
+F 0 "C14" H 8450 2500 50  0000 L CNN
 F 1 "100nF" H 8450 2400 50  0000 L CNN
 F 2 "Capacitor_SMD:C_0603_1608Metric" H 8838 2300 50  0001 C CNN
@@
 $EndComp
 $Comp
-L Device:CP C11
+L Device:CP C15
 U 1 1 6104C514
 P 9050 2450
-F 0 "C11" H 9168 2496 50  0000 L CNN
+F 0 "C15" H 9168 2496 50  0000 L CNN
 F 1 "4.7uF" H 9168 2405 50  0000 L CNN
 F 2 "Capacitor_Tantalum_SMD:CP_EIA-3216-18_Kemet-A" H 9088 2300 50  0001 C CNN
@@
 $EndComp
 $Comp
-L Device:CP C12
+L Device:CP C16
 U 1 1 6104F3B9
 P 10150 2450
-F 0 "C12" H 9850 2500 50  0000 L CNN
+F 0 "C16" H 9850 2500 50  0000 L CNN
 F 1 "4.7uF" H 9850 2400 50  0000 L CNN
 F 2 "Capacitor_Tantalum_SMD:CP_EIA-3216-18_Kemet-A" H 10188 2300 50  0001 C CNN
@@
 $EndComp
 $Comp
-L Device:C C13
+L Device:C C17
 U 1 1 6104FB23
 P 10400 2450
-F 0 "C13" H 10515 2496 50  0000 L CNN
+F 0 "C17" H 10515 2496 50  0000 L CNN
 F 1 "100nF" H 10515 2405 50  0000 L CNN
 F 2 "Capacitor_SMD:C_0603_1608Metric" H 10438 2300 50  0001 C CNN
@@
 $EndComp
 $Comp
-L power:GND #PWR040
+L power:GND #PWR044
 U 1 1 61050D58
 P 8800 2600
-F 0 "#PWR040" H 8800 2350 50  0001 C CNN
+F 0 "#PWR044" H 8800 2350 50  0001 C CNN
 F 1 "GND" H 8805 2427 50  0000 C CNN
 F 2 "" H 8800 2600 50  0001 C CNN
@@
 $EndComp
 $Comp
-L power:GND #PWR041
+L power:GND #PWR045
 U 1 1 610513D3
 P 9050 2600
-F 0 "#PWR041" H 9050 2350 50  0001 C CNN
+F 0 "#PWR045" H 9050 2350 50  0001 C CNN
 F 1 "GND" H 9055 2427 50  0000 C CNN
 F 2 "" H 9050 2600 50  0001 C CNN
@@
 $EndComp
 $Comp
-L power:GND #PWR042
+L power:GND #PWR046
 U 1 1 61051726
 P 10150 2600
-F 0 "#PWR042" H 10150 2350 50  0001 C CNN
+F 0 "#PWR046" H 10150 2350 50  0001 C CNN
 F 1 "GND" H 10155 2427 50  0000 C CNN
 F 2 "" H 10150 2600 50  0001 C CNN
@@
 $EndComp
 $Comp
-L power:GND #PWR043
+L power:GND #PWR047
 U 1 1 61051BAB
 P 10400 2600
-F 0 "#PWR043" H 10400 2350 50  0001 C CNN
+F 0 "#PWR047" H 10400 2350 50  0001 C CNN
 F 1 "GND" H 10405 2427 50  0000 C CNN
 F 2 "" H 10400 2600 50  0001 C CNN
@@
 $EndComp
 $Comp
-L power:GND #PWR039
+L power:GND #PWR043
 U 1 1 61051F07
 P 9600 2550
-F 0 "#PWR039" H 9600 2300 50  0001 C CNN
+F 0 "#PWR043" H 9600 2300 50  0001 C CNN
 F 1 "GND" H 9605 2377 50  0000 C CNN
 F 2 "" H 9600 2550 50  0001 C CNN
@@
 Connection ~ 9050 2250
 $Comp
-L power:+5V #PWR034
+L power:+5V #PWR038
 U 1 1 6105897D
 P 8800 2200
-F 0 "#PWR034" H 8800 2050 50  0001 C CNN
+F 0 "#PWR038" H 8800 2050 50  0001 C CNN
 F 1 "+5V" H 8815 2373 50  0000 C CNN
 F 2 "" H 8800 2200 50  0001 C CNN
@@
 $EndComp
 $Comp
-L power:+3.3V #PWR035
+L power:+3.3V #PWR039
 U 1 1 61059578
 P 10400 2200
-F 0 "#PWR035" H 10400 2050 50  0001 C CNN
+F 0 "#PWR039" H 10400 2050 50  0001 C CNN
 F 1 "+3.3V" H 10415 2373 50  0000 C CNN
 F 2 "" H 10400 2200 50  0001 C CNN
@@
 3.3V LDO regulator
 Text Notes 5000 6150 0    50   ~ 10
-Voltage divider calculations:\n\nU_in max = 8.4V\nU_out max = 3.3V\n\nU_out = U_in * R2/(R1+R2)\nU_out * (R1+R2) = U_in * R2\nU_out * R1+ U_out * R2 = U_in * R2\nU_out * R1 = (U_in - U_out) * R2\nR1 = R2 * (U_in - U_out)/U_out\n\nassume R2 = 10k\n\nR1 = 10000 * (8.4 - 3.3)/3.3 = 15454 ohm -> 16kohm\n
+Voltage divider calculations:\n\nU_in max = 8.4V\nU_out max = 3V\n\nU_out = U_in * R2/(R1+R2)\nU_out * (R1+R2) = U_in * R2\nU_out * R1+ U_out * R2 = U_in * R2\nU_out * R1 = (U_in - U_out) * R2\nR1 = R2 * (U_in - U_out)/U_out\n\nassume R2 = 10k\n\nR1 = 10000 * (8.4 - 3)/3 = 18 kohm\n
 Text Notes 8800 6100 0    50   ~ 10
 Power leds current resistor calculations:\n\ntarget current: I = 5mA\ninput voltage: U1= 3.3V\nforward voltage: Uf = 1.6V\n\nR = (U-Uf)/I\nR_3.3V = (3.3 -1.6)/0.005 = 340 ohm -> 360 ohm
 $Comp
-L Device:CP C14
-U 1 1 60F63913
-P 4100 2550
-F 0 "C14" H 4218 2596 50  0000 L CNN
-F 1 "780uF" H 4218 2505 50  0000 L CNN
-F 2 "Capacitor_THT:CP_Radial_D10.0mm_P5.00mm" H 4138 2400 50  0001 C CNN
-F 3 "~" H 4100 2550 50  0001 C CNN
-	1    4100 2550
-	1    0    0    -1
-$EndComp
-$Comp
-L power:GND #PWR044
-U 1 1 60F63F94
-P 4100 2700
-F 0 "#PWR044" H 4100 2450 50  0001 C CNN
-F 1 "GND" H 4105 2527 50  0000 C CNN
-F 2 "" H 4100 2700 50  0001 C CNN
-F 3 "" H 4100 2700 50  0001 C CNN
-	1    4100 2700
-	1    0    0    -1
-$EndComp
-$Comp
-L Device:C C9
+L Device:C C13
 U 1 1 60FF72EC
 P 6000 2400
-F 0 "C9" H 6115 2446 50  0000 L CNN
+F 0 "C13" H 6115 2446 50  0000 L CNN
 F 1 "33uF" H 6115 2355 50  0000 L CNN
 F 2 "Capacitor_SMD:C_0805_2012Metric" H 6038 2250 50  0001 C CNN
@@
 $EndComp
 $Comp
-L power:GND #PWR037
+L power:GND #PWR041
 U 1 1 60FF77C3
 P 6000 2550
-F 0 "#PWR037" H 6000 2300 50  0001 C CNN
+F 0 "#PWR041" H 6000 2300 50  0001 C CNN
 F 1 "GND" H 6005 2377 50  0000 C CNN
 F 2 "" H 6000 2550 50  0001 C CNN
@@
 $EndComp
 $Comp
-L power:GND #PWR038
+L power:GND #PWR042
 U 1 1 6101E52E
 P 6650 2550
-F 0 "#PWR038" H 6650 2300 50  0001 C CNN
+F 0 "#PWR042" H 6650 2300 50  0001 C CNN
 F 1 "GND" H 6655 2377 50  0000 C CNN
 F 2 "" H 6650 2550 50  0001 C CNN
@@
 $EndComp
 $Comp
-L power:+5V #PWR033
+L power:+5V #PWR037
 U 1 1 61020CAB
 P 7100 2150
-F 0 "#PWR033" H 7100 2000 50  0001 C CNN
+F 0 "#PWR037" H 7100 2000 50  0001 C CNN
 F 1 "+5V" H 7115 2323 50  0000 C CNN
 F 2 "" H 7100 2150 50  0001 C CNN
@@
 Wire Wire Line
 	3550 2350 3600 2350
-Wire Wire Line
-	4100 2350 4100 2400
-Wire Wire Line
-	4100 2350 4150 2350
-Connection ~ 4100 2350
 $Comp
 L Sneak100_kicad:AO4407 Q1
@@
 Connection ~ 3100 2150
 Wire Wire Line
-	3600 2350 4100 2350
+	3600 2350 3650 2350
 Connection ~ 3600 2350
 $EndSCHEMATC

Commit message: component list and values fix
Parts:
- D1: value LED -> RED_LED
Other:
- note added: "Power red led current resistor calculations:\n\ntarget current: I = 5mA\ninput voltage: U1= 3.3V\nforward voltage: Uf = 1.6V\n\nR = (U-Uf)/I\nR_3.3V = (3.3 -1.6)/0.005 = 340 ohm -> 360 ohm"
- note removed: "Power leds current resistor calculations:\n\ntarget current: I = 5mA\ninput voltage: U1= 3.3V\nforward voltage: Uf = 1.6V\n\nR = (U-Uf)/I\nR_3.3V = (3.3 -1.6)/0.005 = 340 ohm -> 360 ohm"
Changed lines of the file:
@@
 P 9550 4650
 F 0 "D1" V 9589 4532 50  0000 R CNN
-F 1 "LED" V 9498 4532 50  0000 R CNN
+F 1 "RED_LED" V 9498 4532 50  0000 R CNN
 F 2 "LED_SMD:LED_0603_1608Metric" H 9550 4650 50  0001 C CNN
 F 3 "~" H 9550 4650 50  0001 C CNN
@@
 Voltage divider calculations:\n\nU_in max = 8.4V\nU_out max = 3V\n\nU_out = U_in * R2/(R1+R2)\nU_out * (R1+R2) = U_in * R2\nU_out * R1+ U_out * R2 = U_in * R2\nU_out * R1 = (U_in - U_out) * R2\nR1 = R2 * (U_in - U_out)/U_out\n\nassume R2 = 10k\n\nR1 = 10000 * (8.4 - 3)/3 = 18 kohm\n
 Text Notes 8800 6100 0    50   ~ 10
-Power leds current resistor calculations:\n\ntarget current: I = 5mA\ninput voltage: U1= 3.3V\nforward voltage: Uf = 1.6V\n\nR = (U-Uf)/I\nR_3.3V = (3.3 -1.6)/0.005 = 340 ohm -> 360 ohm
+Power red led current resistor calculations:\n\ntarget current: I = 5mA\ninput voltage: U1= 3.3V\nforward voltage: Uf = 1.6V\n\nR = (U-Uf)/I\nR_3.3V = (3.3 -1.6)/0.005 = 340 ohm -> 360 ohm
 $Comp
 L Device:C C13

Commit message: Bigger tantalum capacitors
Parts:
- removed C13: 33uF, Capacitor_SMD:C_0805_2012Metric, symbol Device:C
- added C13: 47uF/20V, Capacitor_Tantalum_SMD:CP_EIA-7343-31_Kemet-D, symbol Device:CP
Connections:
- net GND: now also C13.2
- net SUPPLY: now also C13.1
Changed lines of the file:
@@
 Power red led current resistor calculations:\n\ntarget current: I = 5mA\ninput voltage: U1= 3.3V\nforward voltage: Uf = 1.6V\n\nR = (U-Uf)/I\nR_3.3V = (3.3 -1.6)/0.005 = 340 ohm -> 360 ohm
-$Comp
-L Device:C C13
-U 1 1 60FF72EC
-P 6000 2400
-F 0 "C13" H 6115 2446 50  0000 L CNN
-F 1 "33uF" H 6115 2355 50  0000 L CNN
-F 2 "Capacitor_SMD:C_0805_2012Metric" H 6038 2250 50  0001 C CNN
-F 3 "~" H 6000 2400 50  0001 C CNN
-	1    6000 2400
-	1    0    0    -1
-$EndComp
 $Comp
 L power:GND #PWR041
 U 1 1 60FF77C3
-P 6000 2550
-F 0 "#PWR041" H 6000 2300 50  0001 C CNN
-F 1 "GND" H 6005 2377 50  0000 C CNN
-F 2 "" H 6000 2550 50  0001 C CNN
-F 3 "" H 6000 2550 50  0001 C CNN
-	1    6000 2550
+P 5800 2550
+F 0 "#PWR041" H 5800 2300 50  0001 C CNN
+F 1 "GND" H 5805 2377 50  0000 C CNN
+F 2 "" H 5800 2550 50  0001 C CNN
+F 3 "" H 5800 2550 50  0001 C CNN
+	1    5800 2550
 	1    0    0    -1
 $EndComp
-Text GLabel 5950 2200 0    50   Input ~ 0
+Text GLabel 5750 2200 0    50   Input ~ 0
 SUPPLY
 $Comp
@@
 	7100 2200 7100 2150
 Wire Wire Line
-	6250 2200 6000 2200
+	5800 2200 5800 2250
 Wire Wire Line
-	6000 2200 6000 2250
-Wire Wire Line
-	6000 2200 5950 2200
-Connection ~ 6000 2200
+	5800 2200 5750 2200
+Connection ~ 5800 2200
 Wire Wire Line
 	1500 2350 1800 2350
@@
 	3600 2350 3650 2350
 Connection ~ 3600 2350
+$Comp
+L Device:CP C13
+U 1 1 6125F08B
+P 5800 2400
+AR Path="/60E04AFA/6125F08B" Ref="C13"  Part="1"
+AR Path="/60E0499A/6125F08B" Ref="C?"  Part="1"
+F 0 "C13" H 5918 2446 50  0000 L CNN
+F 1 "47uF/20V" H 5918 2355 50  0000 L CNN
+F 2 "Capacitor_Tantalum_SMD:CP_EIA-7343-31_Kemet-D" H 5838 2250 50  0001 C CNN
+F 3 "~" H 5800 2400 50  0001 C CNN
+	1    5800 2400
+	1    0    0    -1
+$EndComp
+Wire Wire Line
+	5800 2200 6250 2200
 $EndSCHEMATC
