File: hardware/sneak100_main_board/power.sch (KiCad schematic (older format))
At the start: 18 parts, among them J5 Conn_01x02, Q1 AO4407, Q2 AO4407, SW1 SW_Push_SPDT, U5 LM1117-3.3, U6 S9V11F5

Commit message: Version 1.1 begin
Changed lines of the file:
@@
 Wire Wire Line
 	3550 2350 3600 2350
-$Comp
-L Sneak100_kicad:AO4407 Q1
-U 1 1 6111B142
-P 2050 2350
-F 0 "Q1" V 2545 2350 50  0000 C CNN
-F 1 "AO4407" V 2450 2350 50  0000 C CNN
-F 2 "Package_SO:SOIC-8_3.9x4.9mm_P1.27mm" H 2550 2500 50  0001 C CNN
-F 3 "" H 2550 2500 50  0001 C CNN
-	1    2050 2350
-	0    -1   -1   0
-$EndComp
 Wire Wire Line
 	2250 2250 2300 2250
@@
 	2300 2150 2300 2250
 Connection ~ 2300 2250
-Wire Wire Line
-	2250 2050 2300 2050
-Wire Wire Line
-	2300 2050 2300 2150
-Connection ~ 2300 2150
 Wire Wire Line
 	1850 2250 1800 2250
@@
 Connection ~ 3100 2250
 Wire Wire Line
-	3150 2050 3100 2050
-Wire Wire Line
-	3100 2050 3100 2150
-Connection ~ 3100 2150
-Wire Wire Line
 	3600 2350 3650 2350
 Connection ~ 3600 2350
@@
 Wire Wire Line
 	5800 2200 6250 2200
+$Comp
+L Sneak100_kicad:AO4407 Q1
+U 1 1 6111B142
+P 2050 2350
+F 0 "Q1" V 2545 2350 50  0000 C CNN
+F 1 "AO4407" V 2450 2350 50  0000 C CNN
+F 2 "Package_SO:SOIC-8_3.9x4.9mm_P1.27mm" H 2550 2500 50  0001 C CNN
+F 3 "" H 2550 2500 50  0001 C CNN
+	1    2050 2350
+	0    -1   -1   0
+$EndComp
+Wire Wire Line
+	1800 2150 1800 2050
+Wire Wire Line
+	1800 2050 1850 2050
+Connection ~ 1800 2150
+Wire Wire Line
+	3600 2150 3600 2050
+Wire Wire Line
+	3600 2050 3550 2050
+Connection ~ 3600 2150
 $EndSCHEMATC

Commit message: Version 1.1 probably finished
Other:
- moved on the sheet: R3, SW1
Changed lines of the file:
@@
 encoding utf-8
 Sheet 3 7
-Title "Sneak100 Main Board V1.0"
-Date "August 2021"
+Title "Sneak100 Main Board V1.1"
+Date "September 2021"
 Rev ""
 Comp ""
@@
 L Device:R R3
 U 1 1 60F4F69A
-P 3350 3000
-F 0 "R3" H 3420 3046 50  0000 L CNN
-F 1 "1k" H 3420 2955 50  0000 L CNN
-F 2 "Resistor_SMD:R_0603_1608Metric" V 3280 3000 50  0001 C CNN
-F 3 "~" H 3350 3000 50  0001 C CNN
-	1    3350 3000
+P 3350 2950
+F 0 "R3" H 3420 2996 50  0000 L CNN
+F 1 "1k" H 3420 2905 50  0000 L CNN
+F 2 "Resistor_SMD:R_0603_1608Metric" V 3280 2950 50  0001 C CNN
+F 3 "~" H 3350 2950 50  0001 C CNN
+	1    3350 2950
 	1    0    0    -1
 $EndComp
@@
 L Switch:SW_Push_SPDT SW1
 U 1 1 60F52713
-P 3050 3350
-F 0 "SW1" H 3600 3400 50  0000 C CNN
-F 1 "SW_Push_SPDT" H 3600 3300 50  0000 C CNN
-F 2 "sneak100_lib:ESP2010_90" H 3050 3350 50  0001 C CNN
-F 3 "~" H 3050 3350 50  0001 C CNN
-	1    3050 3350
+P 3050 3300
+F 0 "SW1" H 3600 3350 50  0000 C CNN
+F 1 "SW_Push_SPDT" H 3600 3250 50  0000 C CNN
+F 2 "sneak100_lib:ESP2010_90" H 3050 3300 50  0001 C CNN
+F 3 "~" H 3050 3300 50  0001 C CNN
+	1    3050 3300
 	-1   0    0    -1
 $EndComp
@@
 	2950 2750 3350 2750
 Wire Wire Line
-	3350 2750 3350 2850
-Wire Wire Line
 	3350 2750 3350 2650
-Connection ~ 3350 2750
 Wire Wire Line
 	2950 2400 2950 2350
@@
 L power:GND #PWR049
 U 1 1 60F78854
-P 2800 3500
-F 0 "#PWR049" H 2800 3250 50  0001 C CNN
-F 1 "GND" H 2805 3327 50  0000 C CNN
-F 2 "" H 2800 3500 50  0001 C CNN
-F 3 "" H 2800 3500 50  0001 C CNN
-	1    2800 3500
-	1    0    0    -1
-$EndComp
-Wire Wire Line
-	2800 3500 2800 3450
-Wire Wire Line
-	2800 3450 2850 3450
+P 2800 3450
+F 0 "#PWR049" H 2800 3200 50  0001 C CNN
+F 1 "GND" H 2805 3277 50  0000 C CNN
+F 2 "" H 2800 3450 50  0001 C CNN
+F 3 "" H 2800 3450 50  0001 C CNN
+	1    2800 3450
+	1    0    0    -1
+$EndComp
+Wire Wire Line
+	2800 3450 2800 3400
+Wire Wire Line
+	2800 3400 2850 3400
 $Comp
 L power:GND #PWR040
@@
 SUPPLY
 Wire Wire Line
-	3250 3350 3350 3350
-Wire Wire Line
-	2850 3250 2800 3250
-Wire Wire Line
-	2800 3250 2800 3200
-Wire Wire Line
-	3350 3150 3350 3200
-Wire Wire Line
-	2800 3200 3350 3200
-Connection ~ 3350 3200
-Wire Wire Line
-	3350 3200 3350 3350
+	3250 3300 3350 3300
+Wire Wire Line
+	2850 3200 2800 3200
+Wire Wire Line
+	2800 3200 2800 3150
+Wire Wire Line
+	3350 3100 3350 3150
+Wire Wire Line
+	2800 3150 3350 3150
+Connection ~ 3350 3150
+Wire Wire Line
+	3350 3150 3350 3300
 $Comp
 L Regulator_Linear:LM1117-3.3 U5
@@
 	3600 2050 3550 2050
 Connection ~ 3600 2150
+Wire Wire Line
+	3350 2800 3350 2750
+Connection ~ 3350 2750
 $EndSCHEMATC
