File: hardware/sneak100_main_board/memory.sch (KiCad schematic (older format))
At the start: 1 part, among them U10 CAT24C256

Commit message: Update gerbers
Other:
- note added: "24C256 eeprom chip"
- note added: "non-volatile memory"
Changed lines of the file:
@@
 Text Notes 6350 4300 0    50   ~ 0
 write protect:\nlow -> normal operation\nhigh -> memory protected against write operations
+Text Notes 4900 2950 0    100  ~ 20
+non-volatile memory
+Text Notes 5300 3100 0    50   ~ 10
+24C256 eeprom chip
 $EndSCHEMATC
