File: hardware/sneak100_main_board/memory.sch (KiCad schematic (older format))
At the start: 1 part, among them U10 CAT24C256

Commit message: Reorganize files
Other:
- note added: "write protect WP:\nlow -> normal operation\nhigh -> memory protected against write operations"
- note removed: "write protect:\nlow -> normal operation\nhigh -> memory protected against write operations"
Changed lines of the file:
@@
 Wire Wire Line
 	6100 3900 6100 3950
-Text HLabel 6050 3800 2    50   Input ~ 0
+Text HLabel 6050 3800 2    50   BiDi ~ 0
 SCL
-Text HLabel 6050 3700 2    50   Input ~ 0
+Text HLabel 6050 3700 2    50   BiDi ~ 0
 SDA
 Text Notes 6350 4300 0    50   ~ 0
-write protect:\nlow -> normal operation\nhigh -> memory protected against write operations
+write protect WP:\nlow -> normal operation\nhigh -> memory protected against write operations
 Text Notes 4900 2950 0    100  ~ 20
 non-volatile memory
