File: hardware/sneak100_main_board_v2/line_board.kicad_sch (KiCad schematic)
At the start: 13 parts, among them J10 Conn_01x06

Commit message: small improvements
Parts:
- R41: renamed from R37; value (none) -> 200
- R42: renamed from R38; value (none) -> 10k
- R43: renamed from R39; value (none) -> 200
- R44: renamed from R40; value (none) -> 10k
- R45: renamed from R41; value (none) -> 200
- R46: renamed from R42; value (none) -> 10k
- R47: renamed from R43; value (none) -> 200
- R48: renamed from R44; value (none) -> 10k
- U15, U16, U17, U18: value (none) -> KTIR0711S
- renumbered J10 to J11
Changed lines of the file:
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@@
   (symbol (lib_id "Device:R") (at 166.37 112.395 180) (unit 1)
     (in_bom yes) (on_board yes)
-    (property "Reference" "R41" (id 0) (at 160.655 111.76 0)
-      (effects (font (size 1.27 1.27)) (justify right))
-    )
-    (property "Value" "" (id 1) (at 160.655 113.665 0)
+    (property "Reference" "R45" (id 0) (at 160.655 111.76 0)
+      (effects (font (size 1.27 1.27)) (justify right))
+    )
+    (property "Value" "200" (id 1) (at 160.655 113.665 0)
       (effects (font (size 1.27 1.27)) (justify right))
     )
@@
   (symbol (lib_id "Connector_Generic:Conn_01x06") (at 222.25 59.055 180) (unit 1)
     (in_bom yes) (on_board yes) (fields_autoplaced)
-    (property "Reference" "J10" (id 0) (at 222.25 45.085 0))
+    (property "Reference" "J11" (id 0) (at 222.25 45.085 0))
     (property "Value" "Conn_01x06" (id 1) (at 222.25 47.625 0))
     (property "Footprint" "" (id 2) (at 222.25 59.055 0)
@@
   (symbol (lib_id "Device:R") (at 248.92 112.395 0) (unit 1)
     (in_bom yes) (on_board yes) (fields_autoplaced)
-    (property "Reference" "R44" (id 0) (at 251.46 111.1249 0)
-      (effects (font (size 1.27 1.27)) (justify left))
-    )
-    (property "Value" "" (id 1) (at 251.46 113.6649 0)
+    (property "Reference" "R48" (id 0) (at 251.46 111.1249 0)
+      (effects (font (size 1.27 1.27)) (justify left))
+    )
+    (property "Value" "10k" (id 1) (at 251.46 113.6649 0)
       (effects (font (size 1.27 1.27)) (justify left))
     )
@@
   (symbol (lib_id "Device:R") (at 184.15 112.395 0) (unit 1)
     (in_bom yes) (on_board yes) (fields_autoplaced)
-    (property "Reference" "R42" (id 0) (at 186.69 111.1249 0)
-      (effects (font (size 1.27 1.27)) (justify left))
-    )
-    (property "Value" "" (id 1) (at 186.69 113.6649 0)
+    (property "Reference" "R46" (id 0) (at 186.69 111.1249 0)
+      (effects (font (size 1.27 1.27)) (justify left))
+    )
+    (property "Value" "10k" (id 1) (at 186.69 113.6649 0)
       (effects (font (size 1.27 1.27)) (justify left))
     )
@@
   (symbol (lib_id "Device:R") (at 53.975 112.395 0) (unit 1)
     (in_bom yes) (on_board yes) (fields_autoplaced)
-    (property "Reference" "R38" (id 0) (at 55.88 111.1249 0)
-      (effects (font (size 1.27 1.27)) (justify left))
-    )
-    (property "Value" "" (id 1) (at 55.88 113.6649 0)
+    (property "Reference" "R42" (id 0) (at 55.88 111.1249 0)
+      (effects (font (size 1.27 1.27)) (justify left))
+    )
+    (property "Value" "10k" (id 1) (at 55.88 113.6649 0)
       (effects (font (size 1.27 1.27)) (justify left))
     )
@@
     (in_bom yes) (on_board yes) (fields_autoplaced)
     (property "Reference" "U15" (id 0) (at 45.085 109.855 0))
-    (property "Value" "" (id 1) (at 45.085 112.395 0))
+    (property "Value" "KTIR0711S" (id 1) (at 45.085 112.395 0))
     (property "Footprint" "" (id 2) (at 45.085 120.015 0)
       (effects (font (size 1.27 1.27)) hide)
@@
     (in_bom yes) (on_board yes) (fields_autoplaced)
     (property "Reference" "U17" (id 0) (at 175.26 109.22 0))
-    (property "Value" "" (id 1) (at 175.26 111.76 0))
+    (property "Value" "KTIR0711S" (id 1) (at 175.26 111.76 0))
     (property "Footprint" "" (id 2) (at 175.26 120.015 0)
       (effects (font (size 1.27 1.27)) hide)
@@
   (symbol (lib_id "Device:R") (at 118.745 112.395 0) (unit 1)
     (in_bom yes) (on_board yes) (fields_autoplaced)
-    (property "Reference" "R40" (id 0) (at 120.65 111.1249 0)
-      (effects (font (size 1.27 1.27)) (justify left))
-    )
-    (property "Value" "" (id 1) (at 120.65 113.6649 0)
+    (property "Reference" "R44" (id 0) (at 120.65 111.1249 0)
+      (effects (font (size 1.27 1.27)) (justify left))
+    )
+    (property "Value" "10k" (id 1) (at 120.65 113.6649 0)
       (effects (font (size 1.27 1.27)) (justify left))
     )
@@
     (in_bom yes) (on_board yes) (fields_autoplaced)
     (property "Reference" "U16" (id 0) (at 109.855 109.22 0))
-    (property "Value" "" (id 1) (at 109.855 111.76 0))
+    (property "Value" "KTIR0711S" (id 1) (at 109.855 111.76 0))
     (property "Footprint" "" (id 2) (at 109.855 120.015 0)
       (effects (font (size 1.27 1.27)) hide)
@@
   (symbol (lib_id "Device:R") (at 100.965 112.395 180) (unit 1)
     (in_bom yes) (on_board yes)
-    (property "Reference" "R39" (id 0) (at 95.25 111.76 0)
-      (effects (font (size 1.27 1.27)) (justify right))
-    )
-    (property "Value" "" (id 1) (at 95.25 113.665 0)
+    (property "Reference" "R43" (id 0) (at 95.25 111.76 0)
+      (effects (font (size 1.27 1.27)) (justify right))
+    )
+    (property "Value" "200" (id 1) (at 95.25 113.665 0)
       (effects (font (size 1.27 1.27)) (justify right))
     )
@@
   (symbol (lib_id "Device:R") (at 231.14 112.395 180) (unit 1)
     (in_bom yes) (on_board yes)
-    (property "Reference" "R43" (id 0) (at 225.425 111.76 0)
-      (effects (font (size 1.27 1.27)) (justify right))
-    )
-    (property "Value" "" (id 1) (at 225.425 113.665 0)
+    (property "Reference" "R47" (id 0) (at 225.425 111.76 0)
+      (effects (font (size 1.27 1.27)) (justify right))
+    )
+    (property "Value" "200" (id 1) (at 225.425 113.665 0)
       (effects (font (size 1.27 1.27)) (justify right))
     )
@@
     (in_bom yes) (on_board yes) (fields_autoplaced)
     (property "Reference" "U18" (id 0) (at 240.03 109.22 0))
-    (property "Value" "" (id 1) (at 240.03 111.76 0))
+    (property "Value" "KTIR0711S" (id 1) (at 240.03 111.76 0))
     (property "Footprint" "" (id 2) (at 240.03 120.015 0)
       (effects (font (size 1.27 1.27)) hide)
@@
   (symbol (lib_id "Device:R") (at 36.195 112.395 180) (unit 1)
     (in_bom yes) (on_board yes)
-    (property "Reference" "R37" (id 0) (at 30.48 111.76 0)
-      (effects (font (size 1.27 1.27)) (justify right))
-    )
-    (property "Value" "" (id 1) (at 30.48 113.665 0)
-      (effects (font (size 1.27 1.27)) (justify right))
-    )
+    (property "Reference" "R41" (id 0) (at 30.48 111.76 0)
+      (effects (font (size 1.27 1.27)) (justify right))
+    )
+    (property "Value" "200" (id 1) (at 30.48 113.665 0)
+      (effects (font (size 1.27 1.27)) (justify right))
+    )
