File: hardware/sneak100_main_board_v2/motors.kicad_sch (KiCad schematic)
At the start: 20 parts

Commit message: PCB version 2.0 schematic progress
Parts:
- C23: renamed from C27; value (none) -> 100nF
- C24: renamed from C29; value (none) -> 100nF
- C25: renamed from C31; value (none) -> 47uF/20V
- C26: renamed from C33; value (none) -> 100nF
- C27: renamed from C35; value (none) -> 100nF
- C28: renamed from C37; value (none) -> 47uF/20V
- C29: renamed from C28; value (none) -> 100nF
- C30: value (none) -> 100nF
- C31: renamed from C32; value (none) -> 47uF/20V
- C32: renamed from C34; value (none) -> 100nF
- C33: renamed from C36; value (none) -> 100nF
- C34: renamed from C38; value (none) -> 47uF/20V
- J6: renamed from J7; value (none) -> Conn_01x06
- U10: renamed from U11; value (none) -> DRV8835
- U7: renamed from U8; value (none) -> DRV8835
- U8: renamed from U10; value (none) -> DRV8835
- U9: value (none) -> DRV8835
- renumbered J9 to J7, J10 to J9

Commit message: small improvements
Parts:
- renumbered J9 to J10, J6 to J7, J7 to J8, J8 to J9
Changed lines of the file:
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@@
   (symbol (lib_id "Connector_Generic:Conn_01x06") (at 127 34.29 0) (unit 1)
     (in_bom yes) (on_board yes)
-    (property "Reference" "J6" (id 0) (at 125.73 22.86 0)
+    (property "Reference" "J7" (id 0) (at 125.73 22.86 0)
       (effects (font (size 1.27 1.27)) (justify left))
     )
@@
   (symbol (lib_id "Connector_Generic:Conn_01x06") (at 127 110.49 0) (unit 1)
     (in_bom yes) (on_board yes)
-    (property "Reference" "J8" (id 0) (at 125.73 99.06 0)
+    (property "Reference" "J9" (id 0) (at 125.73 99.06 0)
       (effects (font (size 1.27 1.27)) (justify left))
     )
@@
   (symbol (lib_id "Connector_Generic:Conn_01x06") (at 255.27 34.29 0) (unit 1)
     (in_bom yes) (on_board yes)
-    (property "Reference" "J7" (id 0) (at 254 22.86 0)
+    (property "Reference" "J8" (id 0) (at 254 22.86 0)
       (effects (font (size 1.27 1.27)) (justify left))
     )
@@
   (symbol (lib_id "Connector_Generic:Conn_01x06") (at 255.27 110.49 0) (unit 1)
     (in_bom yes) (on_board yes)
-    (property "Reference" "J9" (id 0) (at 254 99.06 0)
-      (effects (font (size 1.27 1.27)) (justify left))
-    )
+    (property "Reference" "J10" (id 0) (at 254 99.06 0)
+      (effects (font (size 1.27 1.27)) (justify left))
+    )
