File: hardware/sneak100_main_board_v2/perfs.kicad_sch (KiCad schematic)
At the start: 24 parts, among them SW3 SW_Push, SW4 SW_Push, SW5 SW_Push

Commit message: PCB version 2.0 schematic progress
Parts:
- removed C19, C21, C22, C24: (no value), symbol Device:C
- removed U4: (no value), symbol Sensor_Motion:MPU-6050
- C19: renamed from C20; value (none) -> 100nF
- C20: renamed from C23; value (none) -> 100nF
- C21: renamed from C25; value (none) -> 100nF
- C22: renamed from C26; value (none) -> 4.7uF
- D2: value (none) -> GREEN
- D3: value (none) -> YELLOW
- J5: renamed from J6; value (none) -> Conn_01x06
- R15: renamed from R13; value (none) -> 10k
- R16: renamed from R14; value (none) -> 10k
- R17: renamed from R15; value (none) -> 10k
- R18: renamed from R16; value (none) -> 300
- R19: renamed from R17; value (none) -> 270
- R20: renamed from R18; value (none) -> 100
- U4: renamed from U6; value (none) -> TSOP4838
- U5: value (none) -> CAT24C256
- U6: renamed from U7; value (none) -> SSD1306
- renumbered SW3 to SW4, SW4 to SW5, SW5 to SW6
Connections:
- no-connect marks 2 -> 0
Other:
- note removed: "6DoF IMU"
- moved on the sheet: C22, J5, R20, U4, U5, U6

Commit message: small improvements
Parts:
- renumbered J5 to J6
Changed lines of the file:
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@@
   (symbol (lib_id "Connector_Generic:Conn_01x06") (at 223.52 57.15 180) (unit 1)
     (in_bom yes) (on_board yes) (fields_autoplaced)
-    (property "Reference" "J5" (id 0) (at 223.52 43.18 0))
+    (property "Reference" "J6" (id 0) (at 223.52 43.18 0))
     (property "Value" "Conn_01x06" (id 1) (at 223.52 45.72 0))
     (property "Footprint" "" (id 2) (at 223.52 57.15 0)
