File: hardware/sneak100_main_board_v2/power.kicad_sch (KiCad schematic)
At the start: 21 parts

Commit message: PCB version 2.0 schematic progress
Parts:
- removed J5: (no value), symbol Connector_Generic:Conn_01x04
- added JP1: (no value), symbol Sneak100:jumper_4
- C13: renamed from C15; value (none) -> 100nF
- C14: renamed from C16; value (none) -> 4.7uF
- C15: renamed from C17; value (none) -> 4.7uF
- C16: renamed from C18; value (none) -> 100nF
- C17: renamed from C13; value (none) -> 47uF/20V
- C18: renamed from C14; value (none) -> 100nF
- D1: value (none) -> RED
- J4: value (none) -> Conn_01x02
- Q1, Q2: value (none) -> AO4407
- R10: renamed from R8; value (none) -> 1k
- R11: renamed from R9; value (none) -> 18k
- R12: value (none) -> 360
- R13: renamed from R11; value (none) -> 18k
- R14: renamed from R10; value (none) -> 10k
- R8: renamed from R7; value (none) -> 10k
- R9: renamed from R6; value (none) -> 1k
- SW3: renamed from SW2; value (none) -> SW_Push_SPDT
- U2: renamed from U3; value (none) -> LM1117-3.3
- U3: renamed from U2; value (none) -> S9V11F5
Connections:
- net +5V: now also JP1.4 (B)
- net INPUT: now also JP1.1 (A)
- net STLINK_5V: now also JP1.2 (C), JP1.3 (C)

Commit message: small improvements
Parts:
- removed JP1: (no value), symbol Sneak100:jumper_4
- added J5: (no value), symbol Connector_Generic:Conn_02x03_Odd_Even
Connections:
- net +5V: now also J5.2 (Pin_2), J5.6 (Pin_6)
- net INPUT: now also J4.1 (Pin_1), Q1.5, Q1.6, Q1.7, Q1.8, J5.3 (Pin_3); no longer Q1.1, Q1.2, Q1.3, Q2.1, Q2.2, Q2.3, R8.1
- net STLINK_5V: now also J5.5 (Pin_5)
- new net: Q1.1, Q1.2, Q1.3, Q2.1, Q2.2, Q2.3, R8.1
- new net USB_5V: J5.1 (Pin_1)
- no-connect marks 0 -> 1
Changed lines of the file:
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@@
   (junction (at 54.61 64.77) (diameter 0) (color 0 0 0 0)
   )
+  (junction (at 92.71 137.16) (diameter 0) (color 0 0 0 0)
+  )
   (junction (at 207.01 66.04) (diameter 0) (color 0 0 0 0)
   )
@@
   (junction (at 154.94 135.89) (diameter 0) (color 0 0 0 0)
   )
+  (junction (at 39.37 64.77) (diameter 0) (color 0 0 0 0)
+  )
   (junction (at 139.7 57.15) (diameter 0) (color 0 0 0 0)
   )
@@
   (junction (at 92.71 64.77) (diameter 0) (color 0 0 0 0)
   )
-  (junction (at 69.85 64.77) (diameter 0) (color 0 0 0 0)
-  )
   (junction (at 80.01 62.23) (diameter 0) (color 0 0 0 0)
   )
@@
   (junction (at 92.71 62.23) (diameter 0) (color 0 0 0 0)
   )
-  (junction (at 78.74 139.065) (diameter 0) (color 0 0 0 0)
-  )
   (junction (at 41.91 64.77) (diameter 0) (color 0 0 0 0)
   )
@@
   (junction (at 41.91 62.23) (diameter 0) (color 0 0 0 0)
   )
+  (no_connect (at 91.44 139.7))
   (wire (pts (xy 137.16 135.89) (xy 146.05 135.89))
     (stroke (width 0) (type default) (color 0 0 0 0))
   )
+  (wire (pts (xy 92.71 137.16) (xy 92.71 135.89))
+    (stroke (width 0) (type default) (color 0 0 0 0))
+  )
   (wire (pts (xy 194.31 54.61) (xy 194.31 55.88))
     (stroke (width 0) (type default) (color 0 0 0 0))
@@
     (stroke (width 0) (type default) (color 0 0 0 0))
   )
-  (wire (pts (xy 78.74 141.605) (xy 78.74 139.065))
-    (stroke (width 0) (type default) (color 0 0 0 0))
-  )
   (polyline (pts (xy 180.34 74.93) (xy 120.65 74.93))
     (stroke (width 0) (type default) (color 0 0 0 0))
@@
     (stroke (width 0) (type default) (color 0 0 0 0))
   )
+  (wire (pts (xy 91.44 137.16) (xy 92.71 137.16))
+    (stroke (width 0) (type default) (color 0 0 0 0))
+  )
   (wire (pts (xy 207.01 55.88) (xy 207.01 57.15))
     (stroke (width 0) (type default) (color 0 0 0 0))
@@
     (stroke (width 0) (type default) (color 0 0 0 0))
   )
-  (wire (pts (xy 80.01 139.065) (xy 78.74 139.065))
-    (stroke (width 0) (type default) (color 0 0 0 0))
-  )
   (wire (pts (xy 154.94 135.89) (xy 154.94 137.16))
     (stroke (width 0) (type default) (color 0 0 0 0))
@@
     (stroke (width 0) (type default) (color 0 0 0 0))
   )
-  (wire (pts (xy 78.74 139.065) (xy 77.47 139.065))
-    (stroke (width 0) (type default) (color 0 0 0 0))
-  )
   (wire (pts (xy 236.22 66.04) (xy 250.19 66.04))
     (stroke (width 0) (type default) (color 0 0 0 0))
@@
     (stroke (width 0) (type default) (color 0 0 0 0))
   )
-  (wire (pts (xy 69.85 60.96) (xy 69.85 64.77))
-    (stroke (width 0) (type default) (color 0 0 0 0))
-  )
   (wire (pts (xy 139.7 57.15) (xy 139.7 58.42))
     (stroke (width 0) (type default) (color 0 0 0 0))
@@
     (stroke (width 0) (type default) (color 0 0 0 0))
   )
-  (wire (pts (xy 68.58 60.96) (xy 69.85 60.96))
+  (wire (pts (xy 39.37 53.975) (xy 39.37 64.77))
     (stroke (width 0) (type default) (color 0 0 0 0))
   )
@@
     (stroke (width 0) (type default) (color 0 0 0 0))
   )
+  (wire (pts (xy 91.44 142.24) (xy 92.71 142.24))
+    (stroke (width 0) (type default) (color 0 0 0 0))
+  )
   (wire (pts (xy 80.01 62.23) (xy 81.28 62.23))
     (stroke (width 0) (type default) (color 0 0 0 0))
   )
+  (wire (pts (xy 39.37 64.77) (xy 41.91 64.77))
+    (stroke (width 0) (type default) (color 0 0 0 0))
+  )
+  (wire (pts (xy 35.56 53.975) (xy 39.37 53.975))
+    (stroke (width 0) (type default) (color 0 0 0 0))
+  )
   (wire (pts (xy 76.2 73.66) (xy 76.2 74.93))
     (stroke (width 0) (type default) (color 0 0 0 0))
   )
-  (wire (pts (xy 69.85 64.77) (xy 76.2 64.77))
-    (stroke (width 0) (type default) (color 0 0 0 0))
-  )
-  (wire (pts (xy 36.83 64.77) (xy 41.91 64.77))
+  (wire (pts (xy 36.83 64.77) (xy 39.37 64.77))
     (stroke (width 0) (type default) (color 0 0 0 0))
   )
@@
     (stroke (width 0) (type default) (color 0 0 0 0))
   )
-  (wire (pts (xy 80.01 141.605) (xy 78.74 141.605))
-    (stroke (width 0) (type default) (color 0 0 0 0))
-  )
   (polyline (pts (xy 120.65 130.81) (xy 120.65 110.49))
     (stroke (width 0) (type default) (color 0 0 0 0))
@@
     (stroke (width 0) (type default) (color 0 0 0 0))
   )
-  (wire (pts (xy 83.82 149.225) (xy 83.82 147.955))
-    (stroke (width 0) (type default) (color 0 0 0 0))
-  )
   (wire (pts (xy 41.91 62.23) (xy 43.18 62.23))
     (stroke (width 0) (type default) (color 0 0 0 0))
@@
     (stroke (width 0) (type default) (color 0 0 0 0))
   )
-  (wire (pts (xy 85.09 149.225) (xy 83.82 149.225))
-    (stroke (width 0) (type default) (color 0 0 0 0))
-  )
   (wire (pts (xy 41.91 64.77) (xy 41.91 62.23))
     (stroke (width 0) (type default) (color 0 0 0 0))
@@
     (stroke (width 0) (type default) (color 0 0 0 0))
   )
-  (wire (pts (xy 54.61 64.77) (xy 69.85 64.77))
+  (wire (pts (xy 54.61 64.77) (xy 76.2 64.77))
     (stroke (width 0) (type default) (color 0 0 0 0))
   )
@@
   )
   (wire (pts (xy 73.66 92.71) (xy 73.66 93.98))
+    (stroke (width 0) (type default) (color 0 0 0 0))
+  )
+  (wire (pts (xy 92.71 142.24) (xy 92.71 137.16))
     (stroke (width 0) (type default) (color 0 0 0 0))
   )
@@
     (effects (font (size 2.54 2.54) (thickness 0.508) bold) (justify left bottom))
   )
-  (global_label "STLINK_5V" (shape input) (at 77.47 139.065 180) (fields_autoplaced)
+  (global_label "STLINK_5V" (shape input) (at 78.74 142.24 180) (fields_autoplaced)
     (effects (font (size 1.27 1.27)) (justify right))
-    (property "Intersheet References" "${INTERSHEET_REFS}" (id 0) (at 65.3807 138.9856 0)
+    (property "Intersheet References" "${INTERSHEET_REFS}" (id 0) (at 66.6507 142.1606 0)
       (effects (font (size 1.27 1.27)) (justify right) hide)
     )
@@
     )
   )
-  (global_label "INPUT" (shape input) (at 68.58 60.96 180) (fields_autoplaced)
+  (global_label "INPUT" (shape input) (at 35.56 53.975 180) (fields_autoplaced)
     (effects (font (size 1.27 1.27)) (justify right))
-    (property "Intersheet References" "${INTERSHEET_REFS}" (id 0) (at 60.6636 60.8806 0)
+    (property "Intersheet References" "${INTERSHEET_REFS}" (id 0) (at 27.6436 53.8956 0)
       (effects (font (size 1.27 1.27)) (justify right) hide)
     )
@@
     )
   )
-  (global_label "INPUT" (shape input) (at 85.09 149.225 0) (fields_autoplaced)
-    (effects (font (size 1.27 1.27)) (justify left))
-    (property "Intersheet References" "${INTERSHEET_REFS}" (id 0) (at 93.0064 149.3044 0)
-      (effects (font (size 1.27 1.27)) (justify left) hide)
+  (global_label "INPUT" (shape input) (at 78.74 139.7 180) (fields_autoplaced)
+    (effects (font (size 1.27 1.27)) (justify right))
+    (property "Intersheet References" "${INTERSHEET_REFS}" (id 0) (at 70.8236 139.6206 0)
+      (effects (font (size 1.27 1.27)) (justify right) hide)
     )
   )
@@
     (effects (font (size 1.27 1.27)) (justify right))
     (property "Intersheet References" "${INTERSHEET_REFS}" (id 0) (at 125.0102 57.0706 0)
+      (effects (font (size 1.27 1.27)) (justify right) hide)
+    )
+  )
+  (global_label "USB_5V" (shape input) (at 78.74 137.16 180) (fields_autoplaced)
+    (effects (font (size 1.27 1.27)) (justify right))
+    (property "Intersheet References" "${INTERSHEET_REFS}" (id 0) (at 69.2512 137.0806 0)
       (effects (font (size 1.27 1.27)) (justify right) hide)
     )
@@
     (pin "1")
   )
+  (symbol (lib_id "Connector_Generic:Conn_02x03_Odd_Even") (at 83.82 139.7 0) (unit 1)
+    (in_bom yes) (on_board yes)
+    (property "Reference" "J5" (id 0) (at 85.09 130.175 0))
+    (property "Value" "" (id 1) (at 78.74 132.715 0))
+    (property "Footprint" "" (id 2) (at 83.82 139.7 0)
+      (effects (font (size 1.27 1.27)) hide)
+    )
+    (property "Datasheet" "~" (id 3) (at 83.82 139.7 0)
+      (effects (font (size 1.27 1.27)) hide)
+    )
+    (pin "1")
+    (pin "2")
+    (pin "3")
+    (pin "4")
+    (pin "5")
+    (pin "6")
+  )
   (symbol (lib_id "Device:R") (at 48.26 76.2 0) (unit 1)
     (in_bom yes) (on_board yes) (fields_autoplaced)
@@
     (pin "1")
   )
-  (symbol (lib_id "Sneak100:jumper_4") (at 83.82 140.335 270) (mirror x) (unit 1)
-    (in_bom yes) (on_board yes) (fields_autoplaced)
-    (property "Reference" "JP1" (id 0) (at 85.725 139.0649 90)
-      (effects (font (size 1.27 1.27)) (justify left))
-    )
-    (property "Value" "" (id 1) (at 85.725 141.6049 90)
-      (effects (font (size 1.27 1.27)) (justify left))
-    )
-    (property "Footprint" "" (id 2) (at 83.82 141.605 0)
-      (effects (font (size 1.27 1.27)) hide)
-    )
-    (property "Datasheet" "" (id 3) (at 83.82 141.605 0)
-      (effects (font (size 1.27 1.27)) hide)
-    )
-    (pin "1")
-    (pin "2")
-    (pin "3")
-    (pin "4")
-  )
   (symbol (lib_id "Device:C_Polarized") (at 139.7 62.23 0) (unit 1)
     (in_bom yes) (on_board yes) (fields_autoplaced)
@@
     (pin "2")
   )
-  (symbol (lib_id "power:+5V") (at 83.82 132.715 0) (mirror y) (unit 1)
-    (in_bom yes) (on_board yes) (fields_autoplaced)
-    (property "Reference" "#PWR031" (id 0) (at 83.82 136.525 0)
-      (effects (font (size 1.27 1.27)) hide)
-    )
-    (property "Value" "+5V" (id 1) (at 83.82 127.635 0))
-    (property "Footprint" "" (id 2) (at 83.82 132.715 0)
-      (effects (font (size 1.27 1.27)) hide)
-    )
-    (property "Datasheet" "" (id 3) (at 83.82 132.715 0)
-      (effects (font (size 1.27 1.27)) hide)
-    )
+  (symbol (lib_id "power:+5V") (at 92.71 135.89 0) (mirror y) (unit 1)
+    (in_bom yes) (on_board yes) (fields_autoplaced)
+    (property "Reference" "#PWR031" (id 0) (at 92.71 139.7 0)
+      (effects (font (size 1.27 1.27)) hide)
+    )
+    (property "Value" "+5V" (id 1) (at 92.71 130.81 0))
+    (property "Footprint" "" (id 2) (at 92.71 135.89 0)
+      (effects (font (size 1.27 1.27)) hide)
+    )
+    (property "Datasheet" "" (id 3) (at 92.71 135.89 0)
+      (effects (font (size 1.27 1.27)) hide)
+    )
