File: hardware/sneak100_main_board_v2/proximity.kicad_sch (KiCad schematic)
At the start: 0 parts

Commit message: PCB version 2.0 schematic progress
Parts:
- added C35, C37, C39, C41: (no value), symbol Device:C_Polarized
- added C36, C38, C40, C42: (no value), symbol Device:C
- added C43, C44, C45, C46: 4.7uF, symbol Device:C_Polarized
- added D4, D5, D6, D7: (no value), symbol Device:LED
- added Q3, Q4, Q5, Q6: (no value), symbol Transistor_FET:AO3400A
- added R21, R22, R23, R24, R25, R26, R27, R28, R29, R30, R31, R32: (no value), symbol Device:R
- added R33, R34, R35, R36: 100, symbol Device:R
- added U11, U12, U13, U14: (no value), symbol Interface_Optical:TSOP321xx
Connections:
- new net: D5.2 (A), R22.2
- new net: C44.1, R34.2, U12.2 (Vs)
- new net: D7.1 (K), Q6.3 (D)
- new net: D7.2 (A), R24.2
- new net: Q6.1 (G), R28.2, R32.1
- new net: Q3.1 (G), R25.2, R29.1
- new net: D5.1 (K), Q4.3 (D)
- new net: C43.1, R33.2, U11.2 (Vs)
- new net: C46.1, R36.2, U14.2 (Vs)
- new net: D6.1 (K), Q5.3 (D)
- new net: D6.2 (A), R23.2
- new net: Q5.1 (G), R27.2, R31.1
- new net: Q4.1 (G), R26.2, R30.1
- new net: D4.2 (A), R21.2
- new net: C45.1, R35.2, U13.2 (Vs)
- new net: D4.1 (K), Q3.3 (D)
- new net +3V3: R33.1, R34.1, R35.1, R36.1
- new net +5V: C35.1, C36.1, C37.1, C38.1, C39.1, C40.1, C41.1, C42.1, R21.1, R22.1, R23.1, R24.1
- new net GND: C35.2, C36.2, C37.2, C38.2, C39.2, C40.2, C41.2, C42.2, C43.2, C44.2, C45.2, C46.2, Q3.2 (S), Q4.2 (S), Q5.2 (S), Q6.2 (S), R29.2, R30.2, R31.2, R32.2, U11.3 (GND), U12.3 (GND), U13.3 (GND), U14.3 (GND)
- new net PROX1: U11.1 (OUT)
- new net PROX2: U12.1 (OUT)
- new net PROX3: U13.1 (OUT)
- new net PROX4: U14.1 (OUT)
- new net PROX_GEN: R25.1, R26.1, R27.1, R28.1
Other:
- note added: "PWM frequency: f = 56kHz PWM period: T = 1/f = 17.85us uC pin max current/4: Imax = 5mA uC pin voltage: Uin = 3.3V MOSFET input capacitance: Ciss = 260pF charging: Th = T/2 = 8.9us Rin = 3.3/0.005 = 660 Rin = 680ohm (E24) Ugs = Uin * Rout/(Rin + Rout) = 3.3 * 1000/1680 = 1.964V > 0.7V discharging: Tl = T/2 = 8.9us"
- note added: "diode voltage drop: Ud = 1.3V supply voltage: U = 5V target current: I = 150mA R = (U - Ud)/I R = (5 - 1.3)/0.15 = 3.7/0.15 = 24.66 R = 27ohm (E24)"
- note added: "left-front sensor"
- note added: "left-side sensor"
- note added: "right-front sensor"
- note added: "right-side sensor"

Commit message: small improvements
Parts:
- added D10, D11, D8, D9: (no value), symbol Device:LED
- added R33, R34, R35, R36: (no value), symbol Device:R
- C35, C37, C39, C41: value (none) -> 4.7uF
- C36, C38, C40, C42: value (none) -> 100nF
- D4, D5, D6, D7: value (none) -> IR
- Q3, Q4, Q5, Q6: value (none) -> AO3414; footprint (none) -> Package_TO_SOT_SMD:SOT-23
- R21, R22, R23, R24: value (none) -> 27
- R25, R26, R27, R28: value (none) -> 680
- R29, R30, R31, R32: value (none) -> 1k
- U11, U12, U13, U14: value (none) -> TSOP32156; footprint (none) -> OptoDevice:Vishay_MOLD-3Pin
- renumbered R33 to R37, R34 to R38, R35 to R39, R36 to R40
Connections:
- net +3V3: now also R33.1, R34.1, R35.1, R36.1
- net PROX1: now also D8.1 (K)
- net PROX2: now also D9.1 (K)
- net PROX3: now also D10.1 (K)
- net PROX4: now also D11.1 (K)
- new net: D11.2 (A), R36.2
- new net: D10.2 (A), R35.2
- new net: D8.2 (A), R33.2
- new net: D9.2 (A), R34.2
