File: hardware/sneak100_main_board_v2/sneak100_main_board_v2.kicad_sch (KiCad schematic)
At the start: 0 parts

Commit message: PCB version 2.0 schematic progress
Other:
- added sheet line_board (line_board.kicad_sch)
